Commit message: refactor

File: body.urdf (robot description, URDF)
Before this commit: robot robot, 3 links, 2 joints
Joints:
- joint Torso_FrontLeg: origin xyz=1.5 0 1 rpy=0 0 0 -> xyz=2 0 1 rpy=0 0 0

Commit message: Milestone 4

File: body.urdf (robot description, URDF)
Before this commit: robot robot, 9 links, 8 joints
Joints:
- joint Torso_BackLeg: axis 1 0 0 -> 1 0 1
- joint Torso_FrontLeg: axis 1 0 0 -> 1 0 1
- joint Torso_LeftLeg: axis 0 1 0 -> 0 1 1
- joint Torso_RightLeg: axis 0 1 0 -> 0 1 1
